File: schematics/shield_horiz.brd (EAGLE design)
At the start: 53.3 x 25.4 mm, 10 parts

Commit message: horiz shield update
Routing:
- net VCC: track 65.7 -> 52.5 mm
- net GND: track 64.8 -> 56.5 mm
- net N$6: track 18.5 -> 19.1 mm
Changed lines of the file:
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@@
 <contactref element="JP8" pad="3"/>
 <contactref element="JP9" pad="5"/>
-<wire x1="2.54" y1="5.08" x2="6.985" y2="5.08" width="0.4064" layer="16"/>
-<wire x1="6.985" y1="5.08" x2="11.43" y2="5.08" width="0.4064" layer="16"/>
-<wire x1="11.43" y1="5.08" x2="15.875" y2="5.08" width="0.4064" layer="16"/>
-<wire x1="31.75" y1="6.35" x2="32.385" y2="5.08" width="0.4064" layer="16"/>
-<wire x1="32.385" y1="5.08" x2="31.75" y2="3.81" width="0.4064" layer="16"/>
-<wire x1="31.75" y1="3.81" x2="30.48" y2="2.54" width="0.4064" layer="16"/>
-<wire x1="30.48" y1="2.54" x2="17.78" y2="2.54" width="0.4064" layer="16"/>
-<wire x1="17.78" y1="2.54" x2="17.78" y2="3.175" width="0.4064" layer="16"/>
-<wire x1="17.78" y1="3.175" x2="15.875" y2="5.08" width="0.4064" layer="16"/>
-<wire x1="37.465" y1="5.08" x2="50.8" y2="5.08" width="0.4064" layer="16"/>
-<wire x1="50.8" y1="5.08" x2="32.385" y2="5.08" width="0.4064" layer="16"/>
-<wire x1="46.355" y1="5.08" x2="41.91" y2="5.08" width="0" layer="19" extent="1-1"/>
-<wire x1="37.465" y1="5.08" x2="41.91" y2="5.08" width="0" layer="19" extent="1-1"/>
+<wire x1="2.54" y1="5.08" x2="6.985" y2="5.08" width="0.6096" layer="16"/>
+<wire x1="6.985" y1="5.08" x2="11.43" y2="5.08" width="0.6096" layer="16"/>
+<wire x1="11.43" y1="5.08" x2="15.875" y2="5.08" width="0.6096" layer="16"/>
+<wire x1="37.465" y1="5.08" x2="41.91" y2="5.08" width="0.6096" layer="16"/>
+<wire x1="41.91" y1="5.08" x2="46.355" y2="5.08" width="0.6096" layer="16"/>
+<wire x1="46.355" y1="5.08" x2="46.99" y2="5.08" width="0.6096" layer="16"/>
+<wire x1="46.99" y1="5.08" x2="50.8" y2="5.08" width="0.6096" layer="16"/>
+<wire x1="15.875" y1="5.08" x2="15.875" y2="3.81" width="0.6096" layer="16"/>
+<wire x1="15.875" y1="3.81" x2="31.75" y2="3.81" width="0.6096" layer="16"/>
+<wire x1="31.75" y1="3.81" x2="31.75" y2="6.35" width="0.6096" layer="16"/>
+<wire x1="37.465" y1="5.08" x2="35.56" y2="6.35" width="0.6096" layer="16"/>
+<wire x1="35.56" y1="6.35" x2="31.75" y2="6.35" width="0.6096" layer="16"/>
 </signal>
 <signal name="GND">
@@
 <contactref element="JP8" pad="1"/>
 <contactref element="JP10" pad="1"/>
-<wire x1="2.54" y1="20.32" x2="6.985" y2="20.32" width="0.4064" layer="16"/>
-<wire x1="6.985" y1="20.32" x2="11.43" y2="20.32" width="0.4064" layer="16"/>
-<wire x1="11.43" y1="20.32" x2="15.875" y2="20.32" width="0.4064" layer="16"/>
-<wire x1="15.875" y1="20.32" x2="17.145" y2="20.32" width="0.4064" layer="16"/>
-<wire x1="17.145" y1="20.32" x2="19.05" y2="22.225" width="0.4064" layer="16"/>
-<wire x1="19.05" y1="22.225" x2="30.48" y2="22.225" width="0.4064" layer="16"/>
-<wire x1="30.48" y1="22.225" x2="31.75" y2="20.955" width="0.4064" layer="16"/>
-<wire x1="31.75" y1="20.955" x2="31.75" y2="20.32" width="0.4064" layer="16"/>
-<wire x1="31.75" y1="20.32" x2="31.75" y2="19.05" width="0.4064" layer="16"/>
-<wire x1="37.465" y1="20.32" x2="50.8" y2="20.32" width="0.4064" layer="16"/>
-<wire x1="50.8" y1="20.32" x2="31.75" y2="20.32" width="0.4064" layer="16"/>
-<wire x1="46.355" y1="20.32" x2="41.91" y2="20.32" width="0" layer="19" extent="1-1"/>
-<wire x1="37.465" y1="20.32" x2="41.91" y2="20.32" width="0" layer="19" extent="1-1"/>
+<wire x1="2.54" y1="20.32" x2="6.985" y2="20.32" width="0.6096" layer="16"/>
+<wire x1="6.985" y1="20.32" x2="11.43" y2="20.32" width="0.6096" layer="16"/>
+<wire x1="11.43" y1="20.32" x2="15.875" y2="20.32" width="0.6096" layer="16"/>
+<wire x1="15.875" y1="20.32" x2="18.415" y2="20.32" width="0.6096" layer="16"/>
+<wire x1="18.415" y1="20.32" x2="18.415" y2="21.59" width="0.6096" layer="16"/>
+<wire x1="18.415" y1="21.59" x2="31.75" y2="21.59" width="0.6096" layer="16"/>
+<wire x1="31.75" y1="21.59" x2="31.75" y2="20.32" width="0.6096" layer="16"/>
+<wire x1="31.75" y1="20.32" x2="31.75" y2="19.05" width="0.6096" layer="16"/>
+<wire x1="37.465" y1="20.32" x2="41.91" y2="20.32" width="0.4064" layer="16"/>
+<wire x1="50.8" y1="20.32" x2="46.99" y2="20.32" width="0.6096" layer="16"/>
+<wire x1="46.99" y1="20.32" x2="46.355" y2="20.32" width="0.6096" layer="16"/>
+<wire x1="46.355" y1="20.32" x2="41.91" y2="20.32" width="0.6096" layer="16"/>
+<wire x1="41.91" y1="20.32" x2="31.75" y2="20.32" width="0.6096" layer="16"/>
 </signal>
 <signal name="N$1">
 <contactref element="JP1" pad="2"/>
 <contactref element="JP9" pad="1"/>
-<wire x1="37.465" y1="12.7" x2="26.035" y2="12.7" width="0.4064" layer="16"/>
-<wire x1="26.035" y1="12.7" x2="22.86" y2="10.795" width="0.4064" layer="16"/>
-<wire x1="22.86" y1="10.795" x2="21.59" y2="10.16" width="0.4064" layer="16"/>
-<wire x1="21.59" y1="10.16" x2="21.59" y2="6.35" width="0.4064" layer="16"/>
+<wire x1="37.465" y1="12.7" x2="26.035" y2="12.7" width="0.6096" layer="16"/>
+<wire x1="26.035" y1="12.7" x2="21.59" y2="9.525" width="0.6096" layer="16"/>
+<wire x1="21.59" y1="9.525" x2="21.59" y2="6.35" width="0.6096" layer="16"/>
 </signal>
 <signal name="N$2">
 <contactref element="JP2" pad="2"/>
 <contactref element="JP9" pad="2"/>
-<wire x1="41.91" y1="12.7" x2="41.91" y2="11.43" width="0.4064" layer="16"/>
-<wire x1="41.91" y1="11.43" x2="41.275" y2="10.795" width="0.4064" layer="16"/>
-<wire x1="41.275" y1="10.795" x2="26.035" y2="10.795" width="0.4064" layer="16"/>
-<wire x1="26.035" y1="10.795" x2="24.13" y2="9.525" width="0.4064" layer="16"/>
-<wire x1="24.13" y1="9.525" x2="24.13" y2="6.35" width="0.4064" layer="16"/>
+<wire x1="41.91" y1="12.7" x2="41.91" y2="10.795" width="0.6096" layer="16"/>
+<wire x1="41.91" y1="10.795" x2="26.035" y2="10.795" width="0.6096" layer="16"/>
+<wire x1="26.035" y1="10.795" x2="24.13" y2="9.525" width="0.6096" layer="16"/>
+<wire x1="24.13" y1="9.525" x2="24.13" y2="6.35" width="0.6096" layer="16"/>
 </signal>
 <signal name="N$3">
 <contactref element="JP3" pad="2"/>
 <contactref element="JP9" pad="3"/>
-<wire x1="46.355" y1="12.7" x2="46.99" y2="10.16" width="0.4064" layer="16"/>
-<wire x1="46.99" y1="10.16" x2="46.355" y2="9.525" width="0.4064" layer="16"/>
-<wire x1="46.355" y1="9.525" x2="26.67" y2="9.525" width="0.4064" layer="16"/>
-<wire x1="26.67" y1="9.525" x2="26.67" y2="6.35" width="0.4064" layer="16"/>
+<wire x1="46.355" y1="12.7" x2="46.355" y2="9.525" width="0.6096" layer="16"/>
+<wire x1="46.355" y1="9.525" x2="26.67" y2="9.525" width="0.6096" layer="16"/>
+<wire x1="26.67" y1="9.525" x2="26.67" y2="6.35" width="0.6096" layer="16"/>
 </signal>
 <signal name="N$4">
 <contactref element="JP4" pad="2"/>
 <contactref element="JP9" pad="4"/>
-<wire x1="50.8" y1="12.7" x2="51.435" y2="8.89" width="0.4064" layer="16"/>
-<wire x1="51.435" y1="8.89" x2="50.8" y2="8.255" width="0.4064" layer="16"/>
-<wire x1="50.8" y1="8.255" x2="29.21" y2="8.255" width="0.4064" layer="16"/>
-<wire x1="29.21" y1="8.255" x2="29.21" y2="6.35" width="0.4064" layer="16"/>
+<wire x1="50.8" y1="12.7" x2="50.8" y2="8.255" width="0.6096" layer="16"/>
+<wire x1="50.8" y1="8.255" x2="29.21" y2="8.255" width="0.6096" layer="16"/>
+<wire x1="29.21" y1="8.255" x2="29.21" y2="6.35" width="0.6096" layer="16"/>
 </signal>
 <signal name="N$5">
 <contactref element="JP5" pad="2"/>
 <contactref element="JP10" pad="2"/>
-<wire x1="29.21" y1="19.05" x2="27.305" y2="15.24" width="0.4064" layer="16"/>
-<wire x1="27.305" y1="15.24" x2="22.86" y2="12.7" width="0.4064" layer="16"/>
-<wire x1="22.86" y1="12.7" x2="15.875" y2="12.7" width="0.4064" layer="16"/>
+<wire x1="29.21" y1="19.05" x2="27.305" y2="15.24" width="0.6096" layer="16"/>
+<wire x1="27.305" y1="15.24" x2="20.955" y2="12.7" width="0.6096" layer="16"/>
+<wire x1="20.955" y1="12.7" x2="15.875" y2="12.7" width="0.6096" layer="16"/>
 </signal>
 <signal name="N$6">
 <contactref element="JP6" pad="2"/>
 <contactref element="JP10" pad="3"/>
-<wire x1="26.67" y1="19.05" x2="26.035" y2="16.51" width="0.4064" layer="16"/>
-<wire x1="26.035" y1="16.51" x2="22.225" y2="14.605" width="0.4064" layer="16"/>
-<wire x1="22.225" y1="14.605" x2="13.335" y2="14.605" width="0.4064" layer="16"/>
-<wire x1="13.335" y1="14.605" x2="11.43" y2="12.7" width="0.4064" layer="16"/>
+<wire x1="26.67" y1="19.05" x2="25.4" y2="16.51" width="0.6096" layer="16"/>
+<wire x1="25.4" y1="16.51" x2="20.32" y2="14.605" width="0.6096" layer="16"/>
+<wire x1="20.32" y1="14.605" x2="11.43" y2="14.605" width="0.6096" layer="16"/>
+<wire x1="11.43" y1="14.605" x2="11.43" y2="12.7" width="0.6096" layer="16"/>
 </signal>
 <signal name="N$7">
 <contactref element="JP7" pad="2"/>
 <contactref element="JP10" pad="4"/>
-<wire x1="24.13" y1="19.05" x2="23.495" y2="17.145" width="0.4064" layer="16"/>
-<wire x1="23.495" y1="17.145" x2="22.225" y2="16.51" width="0.4064" layer="16"/>
-<wire x1="22.225" y1="16.51" x2="8.255" y2="16.51" width="0.4064" layer="16"/>
-<wire x1="8.255" y1="16.51" x2="6.985" y2="15.24" width="0.4064" layer="16"/>
-<wire x1="6.985" y1="15.24" x2="6.985" y2="12.7" width="0.4064" layer="16"/>
+<wire x1="24.13" y1="19.05" x2="22.86" y2="17.145" width="0.6096" layer="16"/>
+<wire x1="22.86" y1="17.145" x2="20.955" y2="16.51" width="0.6096" layer="16"/>
+<wire x1="20.955" y1="16.51" x2="6.985" y2="16.51" width="0.6096" layer="16"/>
+<wire x1="6.985" y1="16.51" x2="6.985" y2="12.7" width="0.6096" layer="16"/>
 </signal>
 <signal name="N$8">
@@
 <contactref element="JP10" pad="5"/>
 <wire x1="21.59" y1="19.05" x2="21.59" y2="18.415" width="0.4064" layer="16"/>
-<wire x1="21.59" y1="18.415" x2="20.32" y2="17.78" width="0.4064" layer="16"/>
-<wire x1="20.32" y1="17.78" x2="3.175" y2="17.78" width="0.4064" layer="16"/>
-<wire x1="3.175" y1="17.78" x2="2.54" y2="17.145" width="0.4064" layer="16"/>
-<wire x1="2.54" y1="17.145" x2="2.54" y2="12.7" width="0.4064" layer="16"/>
+<wire x1="21.59" y1="18.415" x2="20.32" y2="17.78" width="0.6096" layer="16"/>
+<wire x1="20.32" y1="17.78" x2="2.54" y2="17.78" width="0.6096" layer="16"/>
+<wire x1="2.54" y1="17.78" x2="2.54" y2="12.7" width="0.6096" layer="16"/>
 </signal>
 </signals>

Commit message: board variant
Routing:
- net GND: track 56.5 -> 52.5 mm
- net N$8: track 24.9 -> 23.0 mm
- net N$4: track 27.9 -> 26.4 mm
- net N$7: track 22.1 -> 20.6 mm
- net N$3: track 26.0 -> 24.7 mm
- net N$2: track 23.2 -> 22.1 mm
- net N$6: track 19.1 -> 18.2 mm
Changed lines of the file:
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@@
 <wire x1="11.43" y1="20.32" x2="15.875" y2="20.32" width="0.6096" layer="16"/>
 <wire x1="15.875" y1="20.32" x2="18.415" y2="20.32" width="0.6096" layer="16"/>
-<wire x1="18.415" y1="20.32" x2="18.415" y2="21.59" width="0.6096" layer="16"/>
-<wire x1="18.415" y1="21.59" x2="31.75" y2="21.59" width="0.6096" layer="16"/>
-<wire x1="31.75" y1="21.59" x2="31.75" y2="20.32" width="0.6096" layer="16"/>
-<wire x1="31.75" y1="20.32" x2="31.75" y2="19.05" width="0.6096" layer="16"/>
-<wire x1="37.465" y1="20.32" x2="41.91" y2="20.32" width="0.4064" layer="16"/>
-<wire x1="50.8" y1="20.32" x2="46.99" y2="20.32" width="0.6096" layer="16"/>
-<wire x1="46.99" y1="20.32" x2="46.355" y2="20.32" width="0.6096" layer="16"/>
+<wire x1="18.415" y1="20.32" x2="20.32" y2="21.59" width="0.6096" layer="16"/>
+<wire x1="20.32" y1="21.59" x2="31.75" y2="21.59" width="0.6096" layer="16"/>
+<wire x1="31.75" y1="21.59" x2="31.75" y2="19.05" width="0.6096" layer="16"/>
+<wire x1="37.465" y1="20.32" x2="41.91" y2="20.32" width="0.6096" layer="16"/>
+<wire x1="50.8" y1="20.32" x2="46.355" y2="20.32" width="0.6096" layer="16"/>
 <wire x1="46.355" y1="20.32" x2="41.91" y2="20.32" width="0.6096" layer="16"/>
-<wire x1="41.91" y1="20.32" x2="31.75" y2="20.32" width="0.6096" layer="16"/>
+<wire x1="31.75" y1="19.05" x2="37.465" y2="19.05" width="0.6096" layer="16"/>
+<wire x1="37.465" y1="19.05" x2="37.465" y2="20.32" width="0.6096" layer="16"/>
 </signal>
 <signal name="N$1">
@@
 <contactref element="JP2" pad="2"/>
 <contactref element="JP9" pad="2"/>
-<wire x1="41.91" y1="12.7" x2="41.91" y2="10.795" width="0.6096" layer="16"/>
-<wire x1="41.91" y1="10.795" x2="26.035" y2="10.795" width="0.6096" layer="16"/>
+<wire x1="41.91" y1="12.7" x2="40.005" y2="10.795" width="0.6096" layer="16"/>
+<wire x1="40.005" y1="10.795" x2="26.035" y2="10.795" width="0.6096" layer="16"/>
 <wire x1="26.035" y1="10.795" x2="24.13" y2="9.525" width="0.6096" layer="16"/>
 <wire x1="24.13" y1="9.525" x2="24.13" y2="6.35" width="0.6096" layer="16"/>
@@
 <contactref element="JP3" pad="2"/>
 <contactref element="JP9" pad="3"/>
-<wire x1="46.355" y1="12.7" x2="46.355" y2="9.525" width="0.6096" layer="16"/>
-<wire x1="46.355" y1="9.525" x2="26.67" y2="9.525" width="0.6096" layer="16"/>
+<wire x1="46.355" y1="12.7" x2="44.45" y2="9.525" width="0.6096" layer="16"/>
+<wire x1="44.45" y1="9.525" x2="26.67" y2="9.525" width="0.6096" layer="16"/>
 <wire x1="26.67" y1="9.525" x2="26.67" y2="6.35" width="0.6096" layer="16"/>
 </signal>
@@
 <contactref element="JP4" pad="2"/>
 <contactref element="JP9" pad="4"/>
-<wire x1="50.8" y1="12.7" x2="50.8" y2="8.255" width="0.6096" layer="16"/>
-<wire x1="50.8" y1="8.255" x2="29.21" y2="8.255" width="0.6096" layer="16"/>
+<wire x1="50.8" y1="12.7" x2="48.895" y2="8.255" width="0.6096" layer="16"/>
+<wire x1="48.895" y1="8.255" x2="29.21" y2="8.255" width="0.6096" layer="16"/>
 <wire x1="29.21" y1="8.255" x2="29.21" y2="6.35" width="0.6096" layer="16"/>
 </signal>
@@
 <wire x1="26.67" y1="19.05" x2="25.4" y2="16.51" width="0.6096" layer="16"/>
 <wire x1="25.4" y1="16.51" x2="20.32" y2="14.605" width="0.6096" layer="16"/>
-<wire x1="20.32" y1="14.605" x2="11.43" y2="14.605" width="0.6096" layer="16"/>
-<wire x1="11.43" y1="14.605" x2="11.43" y2="12.7" width="0.6096" layer="16"/>
+<wire x1="20.32" y1="14.605" x2="12.7" y2="14.605" width="0.6096" layer="16"/>
+<wire x1="12.7" y1="14.605" x2="11.43" y2="12.7" width="0.6096" layer="16"/>
 </signal>
 <signal name="N$7">
@@
 <wire x1="24.13" y1="19.05" x2="22.86" y2="17.145" width="0.6096" layer="16"/>
 <wire x1="22.86" y1="17.145" x2="20.955" y2="16.51" width="0.6096" layer="16"/>
-<wire x1="20.955" y1="16.51" x2="6.985" y2="16.51" width="0.6096" layer="16"/>
-<wire x1="6.985" y1="16.51" x2="6.985" y2="12.7" width="0.6096" layer="16"/>
+<wire x1="20.955" y1="16.51" x2="8.89" y2="16.51" width="0.6096" layer="16"/>
+<wire x1="8.89" y1="16.51" x2="6.985" y2="12.7" width="0.6096" layer="16"/>
 </signal>
 <signal name="N$8">
@@
 <wire x1="21.59" y1="19.05" x2="21.59" y2="18.415" width="0.4064" layer="16"/>
 <wire x1="21.59" y1="18.415" x2="20.32" y2="17.78" width="0.6096" layer="16"/>
-<wire x1="20.32" y1="17.78" x2="2.54" y2="17.78" width="0.6096" layer="16"/>
-<wire x1="2.54" y1="17.78" x2="2.54" y2="12.7" width="0.6096" layer="16"/>
+<wire x1="20.32" y1="17.78" x2="5.08" y2="17.78" width="0.6096" layer="16"/>
+<wire x1="5.08" y1="17.78" x2="2.54" y2="12.7" width="0.6096" layer="16"/>
 </signal>
 </signals>
