File: schematics/shield_horiz_b.brd (EAGLE design)
At the start: 53.3 x 25.4 mm, 10 parts

Commit message: board variant
Parts:
- moved JP8 9.44 mm to (9.53, 19.1), turned to 180 degrees
- moved JP4 9.44 mm to (43.8, 6.35), turned to 0 degrees
- moved JP5 9.44 mm to (9.53, 5.71), turned to 180 degrees
- moved JP1 8.98 mm to (43.8, 19.1), turned to 0 degrees
- moved JP7 3.18 mm to (9.53, 14.6), turned to 180 degrees
- moved JP3 3.17 mm to (43.8, 10.8), turned to 0 degrees
- moved JP6 3.17 mm to (9.53, 10.2), turned to 180 degrees
- moved JP2 2.69 mm to (43.8, 14.6), turned to 0 degrees
Routing:
- net VCC: track 52.6 -> 109.2 mm
- net N$5: track 16.4 -> 54.6 mm
- net N$1: track 20.1 -> 56.5 mm
- net N$6: track 18.5 -> 41.9 mm
- net N$2: track 22.9 -> 45.0 mm
- net GND: track 65.4 -> 49.5 mm
- net N$8: track 24.5 -> 15.9 mm
- net N$7: track 21.7 -> 29.2 mm
- net N$3: track 25.7 -> 33.0 mm
- net N$4: track 27.6 -> 20.4 mm
- added copper zone on layer 16, net N$10
- added copper zone on layer 16, net N$11
- added copper zone on layer 16, net N$19
- added copper zone on layer 16, net N$20
- added copper zone on layer 16, net N$9
