File: schematics/babymidiproto2_shield.brd (EAGLE design)
At the start: 27.9 x 54.3 mm, 10 parts, among them IC1 4051N, K1 6510051365212, U1 TINY85-20-DIP

Commit message: refactor schematic
Parts:
- removed U1: TINY85-20-DIP, manticore-lib:DIP08
- added ATTINY_BABYGNUSBUINO: TINY85-20-DIP, manticore-lib:DIP254P762X533-8
- renumbered IC1 to MULTIPLEXER, K1 to MINIUSB_CONNECTOR, SV8 to PINHEADER_1_4, SV9 to PINHEADER_5_8
Connections:
- net N$10 renamed INPUT_1
- net N$11 renamed INPUT_8
- net N$12 renamed INPUT_7
- net N$13 renamed INPUT_6
- net N$14 renamed INPUT_5
- net N$6 renamed INPUT_4
- net N$7 renamed INPUT_3
- net N$8 renamed INPUT_2
- removed net N$1: R2.2, U1.1
- removed net N$21: MULTIPLEXER.9, U1.3
- removed net N$22: MULTIPLEXER.10, U1.5
- removed net N$23: MULTIPLEXER.11, U1.6
- removed net N$4: R1.2, U1.2
- removed net N$5: MULTIPLEXER.3, U1.7
- new net D_MINUS: ATTINY_BABYGNUSBUINO.1, R2.2
- new net D_PLUS: ATTINY_BABYGNUSBUINO.2, R1.2
- new net MULTIPLEXED_ANALOG_PIN: ATTINY_BABYGNUSBUINO.7, MULTIPLEXER.3
- new net S1: ATTINY_BABYGNUSBUINO.6, MULTIPLEXER.11
- new net S2: ATTINY_BABYGNUSBUINO.5, MULTIPLEXER.10
- new net S3: ATTINY_BABYGNUSBUINO.3, MULTIPLEXER.9
- net GND: now also ATTINY_BABYGNUSBUINO.4; no longer U1.4
- net VCC: now also ATTINY_BABYGNUSBUINO.8; no longer U1.8
Routing:
- net S3: track 0.00 -> 41.3 mm, vias 0 -> 2
- net N$21: track 41.3 -> 0.00 mm, vias 2 -> 0
- net N$5: track 29.0 -> 0.00 mm
- net MULTIPLEXED_ANALOG_PIN: track 0.00 -> 29.0 mm
- net S2: track 0.00 -> 25.7 mm
- net N$22: track 25.7 -> 0.00 mm
- net S1: track 0.00 -> 21.4 mm
- net N$23: track 21.4 -> 0.00 mm
- net GND: track 23.8 -> 16.2 mm
- net N$1: track 5.08 -> 0.00 mm
- net D_MINUS: track 0.00 -> 5.08 mm
- net N$4: track 2.54 -> 0.00 mm
- net D_PLUS: track 0.00 -> 2.54 mm
